File: ZX_Spectrum_i2/ZX_Spectrum_i2.kicad_pcb (KiCad board)
At the start: 2 copper layers, 213.9 x 130.5 mm, 206 parts, among them IC1 DIP-40_W15.24mm, IC10 DIP-16_W7.62mm, IC11 DIP-16_W7.62mm, IC12 DIP-16_W7.62mm, IC13 DIP-16_W7.62mm, IC14 DIP-18_W7.62mm, IC15 DIP-16_W7.62mm, IC16 DIP-16_W7.62mm, IC17 DIP-16_W7.62mm, IC18 DIP-16_W7.62mm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

Commit message: exported PDF with black silkscreen and with green background (KiCad 10)
Other:
- board text added: "2026/03/31"
- board text removed: "2026/03/30"
Changed lines of the file:
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@@
 	)
 	(setup
+		(stackup
+			(layer "F.SilkS"
+				(type "Top Silk Screen")
+			)
+			(layer "F.Paste"
+				(type "Top Solder Paste")
+			)
+			(layer "F.Mask"
+				(type "Top Solder Mask")
+				(thickness 0.01)
+			)
+			(layer "F.Cu"
+				(type "copper")
+				(thickness 0.035)
+			)
+			(layer "dielectric 1"
+				(type "core")
+				(thickness 1.51)
+				(material "FR4")
+				(epsilon_r 4.5)
+				(loss_tangent 0.02)
+			)
+			(layer "B.Cu"
+				(type "copper")
+				(thickness 0.035)
+			)
+			(layer "B.Mask"
+				(type "Bottom Solder Mask")
+				(thickness 0.01)
+			)
+			(layer "B.Paste"
+				(type "Bottom Solder Paste")
+			)
+			(layer "B.SilkS"
+				(type "Bottom Silk Screen")
+			)
+			(copper_finish "None")
+			(dielectric_constraints no)
+		)
 		(pad_to_mask_clearance 0)
 		(allow_soldermask_bridges_in_footprints no)
@@
 		(pcbplotparams
 			(layerselection 0x00000000_00000000_55555555_55555570)
-			(plot_on_all_layers_selection 0x00000000_00000000_00000000_02080021)
+			(plot_on_all_layers_selection 0x00000000_00000000_00000000_02020021)
 			(disableapertmacros no)
 			(usegerberextensions no)
@@
 			(drillshape 2)
 			(scaleselection 1)
-			(outputdirectory "")
+			(outputdirectory "exports/")
 		)
 	)
@@
 		(layer "Edge.Cuts")
 	)
+	(gr_poly
+		(pts
+			(arc
+				(start 168.28 31.61)
+				(mid 169.115032 32.445032)
+				(end 169.950064 31.61)
+			)
+			(xy 169.95 24.01) (xy 254.8 24.01) (xy 254.8 154.51) (xy 40.9 154.51) (xy 40.9 24.01) (xy 168.28 24.01)
+		)
+		(stroke
+			(width 0.05)
+			(type solid)
+		)
+		(fill yes)
+		(layer "User.4")
+	)
 	(image
 		(at 147.863816 89.254606)
-		(layer "Dwgs.User")
+		(layer "Cmts.User")
 		(locked yes)
 		(data "/9j/4AAQSkZJRgABAQIArgCuAAD/2wBDAAoHBwgHBgoICAgLCgoLDhgQDg0NDh0VFhEYIx8lJCIf"
@@
 	(gr_text "ZX Spectrum Issue two mod"
 		(at 186.4 190.6 0)
-		(layer "Cmts.User")
+		(layer "Dwgs.User")
 		(effects
 			(font
@@
 	(gr_text "Copyright 2026 V. Messina"
 		(at 219.6 197.3 0)
-		(layer "Cmts.User")
+		(layer "Dwgs.User")
 		(effects
 			(font
@@
 		)
 	)
-	(gr_text "2026/03/30"
+	(gr_text "2026/03/31"
 		(at 206.9 194.2 0)
-		(layer "Cmts.User")
+		(layer "Dwgs.User")
 		(effects
 			(font
@@
 	(gr_text "0.00.01"
 		(at 268.4 194.3 0)
-		(layer "Cmts.User")
+		(layer "Dwgs.User")
 		(effects
 			(font
